File: CADFiles/PCB/Traffic Control System/Traffic Control System.kicad_pcb (KiCad board)
At the start: 2 copper layers, 30.5 x 36.5 mm, 10 parts, among them J1 Conn_01x04_Pin

Commit message: Update PCB
Routing:
- net Net-(J1-Pin_4): track 47.1 -> 44.2 mm
- net Net-(D3-K): track 16.7 -> 15.7 mm
Other:
- board text added: "GND"
- board text added: "GREEN"
- board text added: "RED"
- board text added: "YELLOW"
Changed lines of the file:
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@@
 			(at 6.3 2.12 0)
 			(layer "F.Fab")
+			(hide yes)
 			(effects
 				(font
@@
 		)
 	)
+	(gr_text "RED\n"
+		(at 44 67.5 270)
+		(layer "F.SilkS")
+		(effects
+			(font
+				(size 0.7 0.45)
+				(thickness 0.1125)
+				(bold yes)
+			)
+			(justify left bottom)
+		)
+	)
+	(gr_text "YELLOW"
+		(at 48 67 270)
+		(layer "F.SilkS")
+		(effects
+			(font
+				(size 0.7 0.45)
+				(thickness 0.1125)
+				(bold yes)
+			)
+			(justify left bottom)
+		)
+	)
+	(gr_text "GND"
+		(at 56.5 67.5 270)
+		(layer "F.SilkS")
+		(effects
+			(font
+				(size 0.7 0.45)
+				(thickness 0.1125)
+				(bold yes)
+			)
+			(justify left bottom)
+		)
+	)
+	(gr_text "GREEN"
+		(at 52 67 270)
+		(layer "F.SilkS")
+		(effects
+			(font
+				(size 0.7 0.45)
+				(thickness 0.1125)
+				(bold yes)
+			)
+			(justify left bottom)
+		)
+	)
+	(segment
+		(start 44.2 40.3)
+		(end 45.5 39)
+		(width 0.6)
+		(layer "F.Cu")
+		(net 1)
+	)
 	(segment
 		(start 44.2 65.5)
@@
 	)
 	(segment
-		(start 44.2 40.3)
-		(end 45.5 39)
-		(width 0.6)
-		(layer "F.Cu")
-		(net 1)
-	)
-	(segment
 		(start 45.5 39)
 		(end 49.21 39)
@@
 	)
 	(segment
-		(start 45 48.5)
-		(end 46 47.5)
-		(width 0.6)
-		(layer "F.Cu")
-		(net 3)
-	)
-	(segment
 		(start 48.4 65.5)
 		(end 45 62.1)
@@
 	)
 	(segment
-		(start 46 47.5)
+		(start 45 62.1)
+		(end 45 48)
+		(width 0.6)
+		(layer "F.Cu")
+		(net 3)
+	)
+	(segment
+		(start 45.5 47.5)
 		(end 49.225 47.5)
 		(width 0.6)
@@
 	)
 	(segment
-		(start 45 62.1)
-		(end 45 48.5)
+		(start 45 48)
+		(end 45.5 47.5)
 		(width 0.6)
 		(layer "F.Cu")
@@
 	)
 	(segment
-		(start 46.016393 56.983607)
-		(end 47 56)
+		(start 45.801 56)
+		(end 49.225 56)
 		(width 0.6)
 		(layer "F.Cu")
@@
 	)
 	(segment
-		(start 49.083607 61.983607)
-		(end 46.016393 61.983607)
+		(start 45.801 58.701)
+		(end 45.801 56)
 		(width 0.6)
 		(layer "F.Cu")
@@
 	(segment
 		(start 52.6 65.5)
-		(end 49.083607 61.983607)
+		(end 45.801 58.701)
 		(width 0.6)
 		(layer "F.Cu")
@@
 	)
 	(segment
-		(start 47 56)
-		(end 49.225 56)
-		(width 0.6)
-		(layer "F.Cu")
-		(net 5)
-	)
-	(segment
-		(start 46.016393 61.983607)
-		(end 46.016393 56.983607)
-		(width 0.6)
-		(layer "F.Cu")
-		(net 5)
-	)
-	(segment
-		(start 56.8 68.899)
-		(end 56.5 69.199)
+		(start 42 68)
+		(end 40.5 66.5)
+		(width 0.6)
+		(layer "F.Cu")
+		(net 6)
+	)
+	(segment
+		(start 56.8 67.2)
+		(end 56 68)
 		(width 0.6)
 		(layer "F.Cu")
@@
 	)
 	(segment
+		(start 56 68)
+		(end 42 68)
+		(width 0.6)
+		(layer "F.Cu")
+		(net 6)
+	)
+	(segment
+		(start 40.5 66.5)
+		(end 40.5 50.5)
+		(width 0.6)
+		(layer "F.Cu")
+		(net 6)
+	)
+	(segment
 		(start 56.8 65.5)
-		(end 56.8 68.899)
-		(width 0.6)
-		(layer "F.Cu")
-		(net 6)
-	)
-	(segment
-		(start 41.5 51.5)
-		(end 40.5 50.5)
-		(width 0.6)
-		(layer "F.Cu")
-		(net 6)
-	)
-	(segment
-		(start 41.5 69)
-		(end 41.5 51.5)
+		(end 56.8 67.2)
 		(width 0.6)
 		(layer "F.Cu")
@@
 		(width 0.6)
 		(layer "F.Cu")
-		(net 6)
-	)
-	(segment
-		(start 56.301 69)
-		(end 41.5 69)
-		(width 0.6)
-		(layer "F.Cu")
-		(net 6)
-	)
-	(segment
-		(start 56.5 69.199)
-		(end 56.301 69)
-		(width 0.6)
-		(layer "F.Cu")
